Commit message: Final

File: ros2_ws/src/umi_rtx_controller/urdf/umi_rtx.urdf (robot description, URDF)
Before this commit: robot umi-rtx, 10 links, 9 joints
Links:
- link base_link: geometry collision box size=1.252 0.132 0.091; visual box size=1.252 0.132 0.091
- link elbow_to_wrist: geometry collision box size=0.252 0.10 0.07; visual box size=0.252 0.10 0.07
- link gripper_base: geometry collision box size=0.077 0.15 0.078; visual box size=0.077 0.15 0.078
- link left_finger: geometry collision box size=0.07 0.015 0.025; visual box size=0.07 0.015 0.025
- link right_finger: geometry collision box size=0.07 0.015 0.025; visual box size=0.07 0.015 0.025
- link shoulder_link: geometry collision box size=0.278 0.132 0.091; visual box size=0.278 0.132 0.091
- link shoulder_to_elbow: geometry collision box size=0.252 0.10 0.10; visual box size=0.252 0.10 0.10
- link wrist_gripper_connection_to_gripper: geometry collision box size=0.10 0.10 0.05; visual box size=0.10 0.10 0.05
- link wrist_to_wrist_gripper_connection: geometry collision box size=0.075 0.10 0.05; visual box size=0.075 0.10 0.05
Joints:
- joint gripper_right: axis 0 1 0  -> 0 1 0
